File: indicators.kicad_sch (KiCad schematic)
At the start: 8 parts

Commit message: Adjusted indicator LEDs * Increased value to decrease brightness and power usage * Increased size to handle heat and make assembly easier
Parts:
- R301, R302, R303, R304: value 1k -> 2k; footprint Resistor_SMD:R_1206_3216Metric -> Resistor_SMD:R_2010_5025Metric
Changed lines of the file:
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@@
     (in_bom yes) (on_board yes) (fields_autoplaced)
     (property "Reference" "R302" (id 0) (at 151.13 73.66 90))
-    (property "Value" "1k" (id 1) (at 151.13 76.2 90))
-    (property "Footprint" "Resistor_SMD:R_1206_3216Metric" (id 2) (at 151.384 78.994 90)
+    (property "Value" "2k" (id 1) (at 151.13 76.2 90))
+    (property "Footprint" "Resistor_SMD:R_2010_5025Metric" (id 2) (at 151.384 78.994 90)
       (effects (font (size 1.27 1.27)) hide)
     )
@@
     (in_bom yes) (on_board yes) (fields_autoplaced)
     (property "Reference" "R303" (id 0) (at 151.13 88.9 90))
-    (property "Value" "1k" (id 1) (at 151.13 91.44 90))
-    (property "Footprint" "Resistor_SMD:R_1206_3216Metric" (id 2) (at 151.384 94.234 90)
+    (property "Value" "2k" (id 1) (at 151.13 91.44 90))
+    (property "Footprint" "Resistor_SMD:R_2010_5025Metric" (id 2) (at 151.384 94.234 90)
       (effects (font (size 1.27 1.27)) hide)
     )
@@
     (in_bom yes) (on_board yes) (fields_autoplaced)
     (property "Reference" "R301" (id 0) (at 151.13 57.15 90))
-    (property "Value" "1k" (id 1) (at 151.13 59.69 90))
-    (property "Footprint" "Resistor_SMD:R_1206_3216Metric" (id 2) (at 151.384 62.484 90)
+    (property "Value" "2k" (id 1) (at 151.13 59.69 90))
+    (property "Footprint" "Resistor_SMD:R_2010_5025Metric" (id 2) (at 151.384 62.484 90)
       (effects (font (size 1.27 1.27)) hide)
     )
@@
     (in_bom yes) (on_board yes) (fields_autoplaced)
     (property "Reference" "R304" (id 0) (at 151.13 104.14 90))
-    (property "Value" "1k" (id 1) (at 151.13 106.68 90))
-    (property "Footprint" "Resistor_SMD:R_1206_3216Metric" (id 2) (at 151.384 109.474 90)
+    (property "Value" "2k" (id 1) (at 151.13 106.68 90))
+    (property "Footprint" "Resistor_SMD:R_2010_5025Metric" (id 2) (at 151.384 109.474 90)
       (effects (font (size 1.27 1.27)) hide)
     )
